Commit message: feat: modularize hand controller with dex-retargeting and yaml config

File: config/robot.urdf (robot description, URDF)
Before this commit: robot lkls73_with_linkerhand_right, 38 links, 37 joints
Links:
- link Body_Base_link: geometry collision mesh filename=package://my_robot/meshes/arm/Body_Base_link.STL; visual mesh filename=package://my_robot/meshes/arm/Body_Base_link.STL
- link Left_Elbow_Pitch_Link: geometry collision mesh filename=package://my_robot/meshes/arm/Left_Elbow_Pitch_Link.STL; visual mesh filename=package://my_robot/meshes/arm/Left_Elbow_Pitch_Link.STL
- link Left_Shoulder_Base_Link: geometry collision mesh filename=package://my_robot/meshes/arm/Left_Shoulder_Base_Link.STL; visual mesh filename=package://my_robot/meshes/arm/Left_Shoulder_Base_Link.STL
- link Left_Shoulder_Pitch_Link: geometry collision mesh filename=package://my_robot/meshes/arm/Left_Shoulder_Pitch_Link.STL; visual mesh filename=package://my_robot/meshes/arm/Left_Shoulder_Pitch_Link.STL
- link Left_Shoulder_Roll_Link: geometry collision mesh filename=package://my_robot/meshes/arm/Left_Shoulder_Roll_Link.STL; visual mesh filename=package://my_robot/meshes/arm/Left_Shoulder_Roll_Link.STL
- link Left_Shoulder_Yaw_Link: geometry collision mesh filename=package://my_robot/meshes/arm/Left_Shoulder_Yaw_Link.STL; visual mesh filename=package://my_robot/meshes/arm/Left_Shoulder_Yaw_Link.STL
- link Left_Wrist_Pitch_Link: geometry collision mesh filename=package://my_robot/meshes/arm/Left_Wrist_Pitch_Link.STL; visual mesh filename=package://my_robot/meshes/arm/Left_Wrist_Pitch_Link.STL
- link Left_Wrist_Roll_Link: geometry collision mesh filename=package://my_robot/meshes/arm/Left_Wrist_Roll_Link.STL; visual mesh filename=package://my_robot/meshes/arm/Left_Wrist_Roll_Link.STL
- link Left_Wrist_Yaw_Link: geometry collision mesh filename=package://my_robot/meshes/arm/Left_Wrist_Yaw_Link.STL; visual mesh filename=package://my_robot/meshes/arm/Left_Wrist_Yaw_Link.STL
- link Right_Elbow_Pitch_Link: geometry collision mesh filename=package://my_robot/meshes/arm/Right_Elbow_Pitch_Link.STL; visual mesh filename=package://my_robot/meshes/arm/Right_Elbow_Pitch_Link.STL
- link Right_Shoulder_Base_Link: geometry collision mesh filename=package://my_robot/meshes/arm/Right_Shoulder_Base_Link.STL; visual mesh filename=package://my_robot/meshes/arm/Right_Shoulder_Base_Link.STL
- link Right_Shoulder_Pitch_Link: geometry collision mesh filename=package://my_robot/meshes/arm/Right_Shoulder_Pitch_Link.STL; visual mesh filename=package://my_robot/meshes/arm/Right_Shoulder_Pitch_Link.STL
- link Right_Shoulder_Roll_Link: geometry collision mesh filename=package://my_robot/meshes/arm/Right_Shoulder_Roll_Link.STL; visual mesh filename=package://my_robot/meshes/arm/Right_Shoulder_Roll_Link.STL
- link Right_Shoulder_Yaw_Link: geometry collision mesh filename=package://my_robot/meshes/arm/Right_Shoulder_Yaw_Link.STL; visual mesh filename=package://my_robot/meshes/arm/Right_Shoulder_Yaw_Link.STL
- link Right_Wrist_Pitch_Link: geometry collision mesh filename=package://my_robot/meshes/arm/Right_Wrist_Pitch_Link.STL; visual mesh filename=package://my_robot/meshes/arm/Right_Wrist_Pitch_Link.STL
- link Right_Wrist_Roll_Link: geometry collision mesh filename=package://my_robot/meshes/arm/Right_Wrist_Roll_Link.STL; visual mesh filename=package://my_robot/meshes/arm/Right_Wrist_Roll_Link.STL
- link Right_Wrist_Yaw_Link: geometry collision mesh filename=package://my_robot/meshes/arm/Right_Wrist_Yaw_Link.STL; visual mesh filename=package://my_robot/meshes/arm/Right_Wrist_Yaw_Link.STL
- link hand_base_link: geometry collision mesh filename=package://my_robot/meshes/hand/hand_base_link.STL; visual mesh filename=package://my_robot/meshes/hand/hand_base_link.STL
- link index_distal: geometry collision mesh filename=package://my_robot/meshes/hand/index_distal.STL; visual mesh filename=package://my_robot/meshes/hand/index_distal.STL
- link index_metacarpals: geometry collision mesh filename=package://my_robot/meshes/hand/index_metacarpals.STL; visual mesh filename=package://my_robot/meshes/hand/index_metacarpals.STL
- link index_middle: geometry collision mesh filename=package://my_robot/meshes/hand/index_middle.STL; visual mesh filename=package://my_robot/meshes/hand/index_middle.STL
- link index_proximal: geometry collision mesh filename=package://my_robot/meshes/hand/index_proximal.STL; visual mesh filename=package://my_robot/meshes/hand/index_proximal.STL
- link middle_distal: geometry collision mesh filename=package://my_robot/meshes/hand/middle_distal.STL; visual mesh filename=package://my_robot/meshes/hand/middle_distal.STL
- link middle_middle: geometry collision mesh filename=package://my_robot/meshes/hand/middle_middle.STL; visual mesh filename=package://my_robot/meshes/hand/middle_middle.STL
- link middle_proximal: geometry collision mesh filename=package://my_robot/meshes/hand/middle_proximal.STL; visual mesh filename=package://my_robot/meshes/hand/middle_proximal.STL
- link pinky_distal: geometry collision mesh filename=package://my_robot/meshes/hand/pinky_distal.STL; visual mesh filename=package://my_robot/meshes/hand/pinky_distal.STL
- link pinky_metacarpals: geometry collision mesh filename=package://my_robot/meshes/hand/pinky_metacarpals.STL; visual mesh filename=package://my_robot/meshes/hand/pinky_metacarpals.STL
- link pinky_middle: geometry collision mesh filename=package://my_robot/meshes/hand/pinky_middle.STL; visual mesh filename=package://my_robot/meshes/hand/pinky_middle.STL
- link pinky_proximal: geometry collision mesh filename=package://my_robot/meshes/hand/pinky_proximal.STL; visual mesh filename=package://my_robot/meshes/hand/pinky_proximal.STL
- link ring_distal: geometry collision mesh filename=package://my_robot/meshes/hand/ring_distal.STL; visual mesh filename=package://my_robot/meshes/hand/ring_distal.STL
- link ring_metacarpals: geometry collision mesh filename=package://my_robot/meshes/hand/ring_metacarpals.STL; visual mesh filename=package://my_robot/meshes/hand/ring_metacarpals.STL
- link ring_middle: geometry collision mesh filename=package://my_robot/meshes/hand/ring_middle.STL; visual mesh filename=package://my_robot/meshes/hand/ring_middle.STL
- link ring_proximal: geometry collision mesh filename=package://my_robot/meshes/hand/ring_proximal.STL; visual mesh filename=package://my_robot/meshes/hand/ring_proximal.STL
- link thumb_distal: geometry collision mesh filename=package://my_robot/meshes/hand/thumb_distal.STL; visual mesh filename=package://my_robot/meshes/hand/thumb_distal.STL
- link thumb_metacarpals: geometry collision mesh filename=package://my_robot/meshes/hand/thumb_metacarpals.STL; visual mesh filename=package://my_robot/meshes/hand/thumb_metacarpals.STL
- link thumb_metacarpals_base1: geometry collision mesh filename=package://my_robot/meshes/hand/thumb_metacarpals_base1.STL; visual mesh filename=package://my_robot/meshes/hand/thumb_metacarpals_base1.STL
- link thumb_metacarpals_base2: geometry collision mesh filename=package://my_robot/meshes/hand/thumb_metacarpals_base2.STL; visual mesh filename=package://my_robot/meshes/hand/thumb_metacarpals_base2.STL
- link thumb_proximal: geometry collision mesh filename=package://my_robot/meshes/hand/thumb_proximal.STL; visual mesh filename=package://my_robot/meshes/hand/thumb_proximal.STL
Joints:
- joint right_arm_hand_fixed_joint: origin xyz=0 0 0 rpy=0 3.14159 0 -> xyz=-0.02 0 -0.055 rpy=0 3.14159 0
