Commit message: vist框架已经在仿真里通过测试，准备集成真机验证

File: config/lkls73_o2_dual_arm_description.urdf (robot description, URDF)
Before this commit: robot lkls73_o2_dual_arm_description, 17 links, 16 joints
Joints:
- joint Right_Elbow_Pitch_Joint: axis 0 1 0 -> 0 -1 0; limit lower=0 upper=2.2 effort=0 velocity=0 -> lower=-2.2 upper=2.2 effort=0 velocity=0
